Commit message: Modifications to facilitate tuning
1. Add a tuner.launch file to include launch of the error_plotter.py
node.
2. Add SIGINT functionality to starter node so that gazebo
physics is paused right before shutdown for tuning consistency.
3. Modify the joint friction value for joint 6 (0.2 -> 0.05) for
better response to torque commands from the program.
4. Error_plotter.py node now shows the plot immediately upon
shutdown request.
5. Modify PD values in pid_junction_node.cpp for joint 6. Further
tuning needed.

File: abb_experimental/abb_irb120_support/urdf/irb120_3_58_macro.xacro (robot description, xacro)
@@ -199,5 +199,5 @@
       <limit effort="900" lower="-6.98132" upper="6.98132" velocity="7.33038"/>
       <axis xyz="1 0 0"/>
-      <dynamics damping="0.0" friction="0.2"/>
+      <dynamics damping="0.0" friction="0.05"/>
     </joint>
     <!-- end of joint list -->
